File: PCB/ReadCO2/ReadCO2.sch (KiCad schematic (older format))
At the start: 6 parts, among them J1 Conn_01x05, J2 Conn_01x03, J3 Conn_01x04

Commit message: edited PCB
edited pcb layout to fit Eckers case idea
Connections:
- net light_sense: now also A1.26 (A7); no longer A1.19 (A0)
Changed lines of the file:
@@
 Text GLabel 1250 1550 2    50   Input ~ 0
 CO2TX_uCRX
-Text GLabel 6900 2800 2    50   Input ~ 0
+Text GLabel 6900 3500 2    50   Input ~ 0
 light_sense
 Text GLabel 5900 2400 0    50   Input ~ 0
